File: Electronique/prototype_1/prototype_1.kicad_sch (KiCad schematic)
At the start: 3 parts, among them U1 WeMos_D1_mini, U2 L298N, U3 TSOP21xx

Commit message: Mise à jour pour le schéma
Parts:
- removed U2: L298N, Package_TO_SOT_THT:TO-220-15_P2.54x2.54mm_StaggerOdd_Lead4.58mm_Vertical, symbol Driver_Motor:L298N
- added M1, M2: Motor_DC, symbol Motor:Motor_DC
- added SW1: L9110S, symbol MyLibrary:L9110S
Connections:
- net +5V: now also SW1. (VCC); no longer U1.9 (5V), U3.2 (Vs)
- net Earth: now also SW1. (VCC); no longer U1.10 (GND), U3.3 (GND)
- net at U1.12 (D3): now also SW1. (VCC)
- net at U1.14 (SCL/D1): now also SW1. (VCC)
- net +3V3: no longer names the net of U1.8 (3V3)
- net Moteur1 renamed MoteurA
- net MoteurA: now also SW1. (VCC)
- net Moteur2 renamed MoteurB
- net MoteurB: now also SW1. (VCC)
- new net: M1.1 (+), SW1.1 (MotorA-A)
- new net: M1.2 (-), SW1.2 (MotorB-A)
- new net: M2.1 (+), SW1.3 (MotorA-B)
- new net: M2.2 (-), SW1.4 (MotorB-B)
- new net GND: U1.10 (GND)
- no-connect marks 8 -> 9
